File: Kicad/ElectronULA - MAX 10 Board V1.04/ElectronULA.kicad_pcb (KiCad board)
At the start: 4 copper layers, 49 x 68.4 mm, 77 parts, among them J1 Conn_01x02, J2 Micro_SD_Card_Det_Hirose_DM3AT, SW1 SW_DIP_x04, U1 10M08SCE144C8G, U10 SN74HCT125D, U2 74LVC4245APW, U3 74LVC4245APW, U4 74LVC4245APW, U5 74LVC4245APW, U6 74LVC4245APW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

Commit message: Updated with latest VHDL and Kicad Ver 1.05 Board
Routing:
- net /5V: track 165.9 -> 183.3 mm, vias 9 -> 11
