File: Kicad/ElectronULA - MAX 10 Board V1.05/ElectronULA.kicad_pcb (KiCad board)
At the start: 4 copper layers, 49 x 68.4 mm, 89 parts, among them J1 Conn_01x02, J2 Micro_SD_Card_Det_Hirose_DM3AT, SW1 SW_DIP_x04, U1 10M08SCE144C8G, U10 ELECTRON_ULA_PGA_68, U2 SN74HCT125D, U3 74LVC4245APW, U4 74LVC4245APW, U5 74LVC4245APW, U6 74LVC4245APW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

Commit message: Update Gerbers
Routing:
- net /PD_DIR: track 30.2 -> 30.8 mm
Changed lines of the file:
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@@
     (property "ki_keywords" "ULA")
     (attr through_hole)
-    (fp_text reference "U10" (at -0.7711 -5.0151) (layer "F.SilkS")
+    (fp_text reference "U10" (at -0.0201 -1.6411) (layer "F.SilkS")
         (effects (font (size 1 1) (thickness 0.15)))
     )
@@
     (property "ki_keywords" "capacitor cap")
     (attr smd)
-    (fp_text reference "C1" (at -1.908 1.285) (layer "B.SilkS")
+    (fp_text reference "C1" (at -0.027 -1.473) (layer "B.SilkS")
         (effects (font (size 1 1) (thickness 0.15)) (justify mirror))
     )
@@
     (property "ki_keywords" "capacitor cap")
     (attr smd)
-    (fp_text reference "C13" (at 0.93726 2.23266 180) (layer "B.SilkS")
+    (fp_text reference "C13" (at 0.35608 2.1531 180) (layer "B.SilkS")
         (effects (font (size 1 1) (thickness 0.15)) (justify mirror))
     )
@@
     (property "ki_keywords" "capacitor cap")
     (attr smd)
-    (fp_text reference "C18" (at -0.00508 -1.62814) (layer "B.SilkS")
+    (fp_text reference "C18" (at 0.06962 -1.6299) (layer "B.SilkS")
         (effects (font (size 1 1) (thickness 0.15)) (justify mirror))
     )
@@
     (property "ki_keywords" "R res resistor")
     (attr smd)
-    (fp_text reference "R28" (at 2.7432 -0.00508 90) (layer "B.SilkS")
+    (fp_text reference "R28" (at 2.992 0.04948 90) (layer "B.SilkS")
         (effects (font (size 1 1) (thickness 0.15)) (justify mirror))
     )
@@
     (property "ki_keywords" "R res resistor")
     (attr smd)
-    (fp_text reference "R29" (at 2.67716 -0.02032 90) (layer "B.SilkS")
+    (fp_text reference "R29" (at 2.88856 0.01848 90) (layer "B.SilkS")
         (effects (font (size 1 1) (thickness 0.15)) (justify mirror))
     )
@@
     (property "ki_keywords" "R res resistor")
     (attr smd)
-    (fp_text reference "R27" (at 3.26644 -0.04572 90) (layer "B.SilkS")
+    (fp_text reference "R27" (at 2.98704 0.04728 90) (layer "B.SilkS")
         (effects (font (size 1 1) (thickness 0.15)) (justify mirror))
     )
@@
     (property "ki_keywords" "capacitor cap")
     (attr smd)
-    (fp_text reference "C11" (at -2.29616 -0.1143 180) (layer "B.SilkS")
+    (fp_text reference "C11" (at -0.30916 -1.92236 180) (layer "B.SilkS")
         (effects (font (size 1 1) (thickness 0.15)) (justify mirror))
     )
@@
     (property "ki_keywords" "capacitor cap")
     (attr smd)
-    (fp_text reference "C10" (at -0.04318 -1.28778) (layer "B.SilkS")
+    (fp_text reference "C10" (at -0.27606 -1.22434) (layer "B.SilkS")
         (effects (font (size 1 1) (thickness 0.15)) (justify mirror))
     )
@@
     (property "ki_keywords" "R res resistor")
     (attr smd)
-    (fp_text reference "R8" (at 3.43408 0) (layer "B.SilkS")
+    (fp_text reference "R8" (at 3.05504 -0.032) (layer "B.SilkS")
         (effects (font (size 1 1) (thickness 0.15)) (justify mirror))
     )
@@
     (property "ki_keywords" "cap capacitor")
     (attr smd)
-    (fp_text reference "C27" (at 0 -2.3368 180) (layer "B.SilkS")
+    (fp_text reference "C27" (at 0.0118 2.4624 180) (layer "B.SilkS")
         (effects (font (size 1 1) (thickness 0.15)) (justify mirror))
     )
@@
     (property "ki_keywords" "capacitor cap")
     (attr smd)
-    (fp_text reference "C31" (at 0 1.43 90) (layer "B.SilkS")
+    (fp_text reference "C31" (at -0.033 1.919 180) (layer "B.SilkS")
         (effects (font (size 1 1) (thickness 0.15)) (justify mirror))
     )
@@
     (effects (font (size 1 1) (thickness 0.15)))
   )
-  (gr_text "Electron ULA - V1.05" (at 177.4242 86.51 90) (layer "F.SilkS")
+  (gr_text "Electron ULA - V1.05" (at 177.6412 86.493 90) (layer "F.SilkS")
     (effects (font (size 1 1) (thickness 0.125)))
   )
@@
   (segment (start 173.3742 99.057) (end 173.3862 99.069) (width 0.102) (layer "B.Cu") (net 67))
   (segment (start 166.1442 72.851) (end 171.3452 78.052) (width 0.102) (layer "B.Cu") (net 67))
-  (segment (start 170.7802 103.111) (end 170.7802 102.761) (width 0.102) (layer "F.Cu") (net 68))
+  (segment (start 170.7802 103.111) (end 170.7802 101.739) (width 0.102) (layer "F.Cu") (net 68))
   (segment (start 161.8872 81.291) (end 161.8872 80.03062) (width 0.102) (layer "F.Cu") (net 68))
+  (segment (start 170.2852 101.244) (end 168.7972 101.244) (width 0.102) (layer "F.Cu") (net 68))
   (segment (start 161.8872 80.03062) (end 161.88182 80.02524) (width 0.102) (layer "F.Cu") (net 68))
-  (segment (start 169.2632 101.244) (end 168.7972 101.244) (width 0.102) (layer "F.Cu") (net 68))
-  (segment (start 170.7802 102.761) (end 169.2632 101.244) (width 0.102) (layer "F.Cu") (net 68))
+  (segment (start 170.7802 101.739) (end 170.2852 101.244) (width 0.102) (layer "F.Cu") (net 68))
   (via (at 161.88182 80.02524) (size 0.8) (drill 0.4) (layers "F.Cu" "B.Cu") (net 68))
   (via (at 168.7972 101.244) (size 0.8) (drill 0.4) (layers "F.Cu" "B.Cu") (net 68))
